File: SCH_PCB/CANDY/CANDY01A/CANDY01A.sch (KiCad schematic (older format))
At the start: 34 parts, among them J1 HEADER_2x04_PARALLEL, M1 HOLE, M2 HOLE, M3 HOLE, M4 HOLE

Commit message: Edit schema
Parts:
- D3: renamed from D?; value REFERENCE -> LM4041AIM3-1.2/NOP
- Q1: renamed from Q?; value Q_NMOS_GSD -> BSS138
- U1: renamed from U?; value OZ -> OPA2314
- U2, U3: renamed from U?; value OPA2340 -> OPA2314
- gave numbers to parts that had none: 22
Connections:
- net at C7.1, R7.1, U2.1: now also U2.5 (+); no longer U2.3 (+)
- net at D4.2 (A): now also U2.7; no longer U2.1
- net at R8.2: now also U2.6 (-); no longer U2.2 (-)

Commit message: revise of schematic
Parts:
- removed D5: D, symbol D
- added C5: 1 uF, symbol C
- added R10: 39, symbol R
- C5: value 12pF -> 1 pF
- C7: value 1nF -> 1 nF
- D1: symbol DIODE -> DIODE-RESCUE-CANDY01A
- D2: value D_Photo -> PIN
- D4: value D -> 1N4148
- R3, R6: value 1k -> 0
- R5: value 1k -> 3k3
- renumbered R10 to R11
Connections:
- wire segments 79 -> 84
Other:
- note removed: "22x\n7kHz"
- moved on the sheet: BT1, C4, C5, C6, C7, C8, D2, D4, Q1, R11, R3, R4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

Commit message: Data editing
update schema, new label
Parts:
- added R6: 1k, symbol R
- C4: value 100nF -> 4u7
- C8: renamed from C7; value 1 nF -> 2n2
- D2: value PIN -> PIN - S2744-09
- R11: renamed from R10; value 39 -> 51
- renumbered C5 to C6, C6 to C7, C8 to C9, R9 to R10, R11 to R12, R6 to R7, R7 to R8, R8 to R9, U2 to U1, U3 to U2
Changed lines of the file:
@@
 EESchema Schematic File Version 2
-LIBS:CANDY01A-rescue
+LIBS:MLAB_BATERY
+LIBS:MLAB_CONNECTORS
+LIBS:MLAB_D
+LIBS:MLAB_DISPLAY
+LIBS:MLAB_IO
+LIBS:MLAB_Jumpers
+LIBS:MLAB_SW
+LIBS:MLAB_T
+LIBS:MLAB_U
 LIBS:74xgxx
 LIBS:74xx
@@
 LIBS:microchip_pic32mcu
 LIBS:microcontrollers
+LIBS:mlab_header
+LIBS:mlab_mechanical
 LIBS:motor_drivers
 LIBS:motorola
@@
 LIBS:Zilog
 LIBS:CANDY01A-cache
-EELAYER 25 0
+EELAYER 26 0
 EELAYER END
 $Descr A4 11693 8268
@@
 P 2500 3300
 F 0 "D2" H 2450 3595 50  0000 C CNN
-F 1 "PIN" H 2450 3504 50  0000 C CNN
+F 1 "PIN - S2744-09" H 2450 3504 50  0000 C CNN
 F 2 "" H 750 350 50  0001 C CNN
 F 3 "" H 750 350 50  0001 C CNN
@@
 P 3000 4150
 F 0 "C4" H 3115 4196 50  0000 L CNN
-F 1 "100nF" H 3115 4105 50  0000 L CNN
+F 1 "4u7" H 3115 4105 50  0000 L CNN
 F 2 "" H 588 350 50  0001 C CNN
 F 3 "" H 550 500 50  0001 C CNN
@@
 $EndComp
 $Comp
-L OPA2340 U2
-U 1 1 58E3AD53
+L OPA2340 U1
+U 2 1 58E3AD53
 P 6000 3500
-F 0 "U2" H 6100 3700 50  0000 L CNN
+F 0 "U1" H 6100 3700 50  0000 L CNN
 F 1 "OPA2314" H 6050 3250 50  0000 L CNN
 F 2 "" H 3750 300 50  0001 C CNN
 F 3 "" H 3850 200 50  0001 C CNN
-	1    6000 3500
+	2    6000 3500
 	1    0    0    1
 $EndComp
 $Comp
-L R R6
+L R R7
 U 1 1 58E3BCF2
 P 5600 3850
-F 0 "R6" V 5500 3850 50  0000 C CNN
+F 0 "R7" V 5500 3850 50  0000 C CNN
 F 1 "0" V 5600 3850 50  0000 C CNN
 F 2 "" V 1330 950 50  0001 C CNN
@@
 $EndComp
 $Comp
-L R R7
+L R R8
 U 1 1 58E3BE3A
 P 6100 2650
-F 0 "R7" V 6000 2650 50  0000 C CNN
+F 0 "R8" V 6000 2650 50  0000 C CNN
 F 1 "22k" V 6100 2650 50  0000 C CNN
 F 2 "" V 1830 -250 50  0001 C CNN
@@
 $EndComp
 $Comp
-L C C7
+L C C8
 U 1 1 58E3C0E9
 P 6100 2300
-F 0 "C7" V 5950 2300 50  0000 C CNN
-F 1 "1 nF" V 6250 2300 50  0000 C CNN
+F 0 "C8" V 5950 2300 50  0000 C CNN
+F 1 "2n2" V 6250 2300 50  0000 C CNN
 F 2 "" H 3688 -1500 50  0001 C CNN
 F 3 "" H 3650 -1350 50  0001 C CNN
@@
 $EndComp
 $Comp
-L C C6
+L C C7
 U 1 1 58E3C16D
 P 5600 4250
-F 0 "C6" V 5450 4250 50  0000 C CNN
+F 0 "C7" V 5450 4250 50  0000 C CNN
 F 1 "4uF" V 5750 4250 50  0000 C CNN
 F 2 "" H 3188 450 50  0001 C CNN
@@
 $Comp
 L OPA2340 U2
-U 2 1 58E3C1FE
+U 1 1 58E3C1FE
 P 7250 3400
 F 0 "U2" H 7350 3600 50  0000 L CNN
@@
 F 2 "" H 5000 200 50  0001 C CNN
 F 3 "" H 5100 100 50  0001 C CNN
-	2    7250 3400
+	1    7250 3400
 	1    0    0    1
 $EndComp
 $Comp
-L R R8
+L R R9
 U 1 1 58E3C2A4
 P 7250 2650
-F 0 "R8" V 7150 2650 50  0000 C CNN
+F 0 "R9" V 7150 2650 50  0000 C CNN
 F 1 "1k" V 7250 2650 50  0000 C CNN
 F 2 "" V 2980 -250 50  0001 C CNN
@@
 $EndComp
 $Comp
-L R R9
+L R R10
 U 1 1 58E3C574
 P 8200 3400
-F 0 "R9" V 8100 3400 50  0000 C CNN
+F 0 "R10" V 8100 3400 50  0000 C CNN
 F 1 "100" V 8200 3400 50  0000 C CNN
 F 2 "" V 3930 500 50  0001 C CNN
@@
 $EndComp
 $Comp
-L C C8
+L C C9
 U 1 1 58E3C609
 P 8450 3600
-F 0 "C8" V 8300 3600 50  0000 C CNN
+F 0 "C9" V 8300 3600 50  0000 C CNN
 F 1 "1nF" V 8600 3600 50  0000 C CNN
 F 2 "" H 6038 -200 50  0001 C CNN
@@
 $EndComp
 $Comp
-L OPA2340 U3
-U 1 1 58E3C87D
+L OPA2340 U2
+U 2 1 58E3C87D
 P 9300 3300
-F 0 "U3" H 9400 3500 50  0000 L CNN
+F 0 "U2" H 9400 3500 50  0000 L CNN
 F 1 "OPA2314" H 9350 3050 50  0000 L CNN
 F 2 "" H 7050 100 50  0001 C CNN
 F 3 "" H 7150 0   50  0001 C CNN
-	1    9300 3300
+	2    9300 3300
 	1    0    0    1
 $EndComp
@@
 	3550 2300 3800 2300
 Wire Wire Line
-	5600 3400 5700 3400
+	5300 3400 5700 3400
 $Comp
 L GND #PWR12
@@
 	8800 4600 8800 4700
 $Comp
-L R R11
+L R R12
 U 1 1 58E46236
 P 9300 4400
-F 0 "R11" V 9200 4400 50  0000 C CNN
+F 0 "R12" V 9200 4400 50  0000 C CNN
 F 1 "10k" V 9300 4400 50  0000 C CNN
 F 2 "" V 5030 1500 50  0001 C CNN
@@
 $EndComp
 $Comp
-L C C5
+L C C6
 U 1 1 59ADCC84
 P 4050 3400
-F 0 "C5" V 3900 3400 50  0000 C CNN
+F 0 "C6" V 3900 3400 50  0000 C CNN
 F 1 "1 uF" V 4200 3400 50  0000 C CNN
 F 2 "" H 1638 -400 50  0001 C CNN
@@
 REF
 $Comp
-L R R10
+L R R11
 U 1 1 59ADE06B
 P 8800 3850
-F 0 "R10" V 8593 3850 50  0000 C CNN
-F 1 "39" V 8684 3850 50  0000 C CNN
+F 0 "R11" V 8593 3850 50  0000 C CNN
+F 1 "51" V 8684 3850 50  0000 C CNN
 F 2 "" V 4530 950 50  0001 C CNN
 F 3 "" H 4600 950 50  0001 C CNN
@@
 	4700 4150 4650 4150
 Wire Wire Line
-	5600 3450 5600 3400
-Wire Wire Line
-	5650 3400 4200 3400
-Wire Wire Line
 	4700 3700 4700 3400
 Connection ~ 4700 3400
+$Comp
+L R R6
+U 1 1 59D66B3F
+P 5150 3400
+F 0 "R6" V 5050 3400 50  0000 C CNN
+F 1 "1k" V 5150 3400 50  0000 C CNN
+F 2 "" V 880 500 50  0001 C CNN
+F 3 "" H 950 500 50  0001 C CNN
+	1    5150 3400
+	0    -1   -1   0
+$EndComp
+Wire Wire Line
+	4200 3400 5000 3400
+Wire Wire Line
+	5900 3850 5900 3800
 $EndSCHEMATC

Commit message: change schematics R11/D5 R12
Parts:
- removed R11: 51, symbol R
- added D5: 1N4148, symbol D
- R12: value 10k -> 120M
Connections:
- net at C9.2, R10.1, U2.5 (+): now also D5.2 (A)
- net at Q1.3 (D): now also D5.1 (K)
Changed lines of the file:
@@
 EESchema Schematic File Version 2
-LIBS:MLAB_BATERY
-LIBS:MLAB_CONNECTORS
-LIBS:MLAB_D
-LIBS:MLAB_DISPLAY
-LIBS:MLAB_IO
-LIBS:MLAB_Jumpers
-LIBS:MLAB_SW
-LIBS:MLAB_T
-LIBS:MLAB_U
 LIBS:74xgxx
 LIBS:74xx
@@
 LIBS:microchip_pic32mcu
 LIBS:microcontrollers
-LIBS:mlab_header
-LIBS:mlab_mechanical
 LIBS:motor_drivers
 LIBS:motorola
@@
 LIBS:Zilog
 LIBS:CANDY01A-cache
-EELAYER 26 0
+EELAYER 25 0
 EELAYER END
 $Descr A4 11693 8268
@@
 P 9300 4400
 F 0 "R12" V 9200 4400 50  0000 C CNN
-F 1 "10k" V 9300 4400 50  0000 C CNN
+F 1 "120M" V 9300 4400 50  0000 C CNN
 F 2 "" V 5030 1500 50  0001 C CNN
 F 3 "" H 5100 1500 50  0001 C CNN
@@
 Text Label 4650 4200 2    60   ~ 0
 REF
-$Comp
-L R R11
-U 1 1 59ADE06B
-P 8800 3850
-F 0 "R11" V 8593 3850 50  0000 C CNN
-F 1 "51" V 8684 3850 50  0000 C CNN
-F 2 "" V 4530 950 50  0001 C CNN
-F 3 "" H 4600 950 50  0001 C CNN
-	1    8800 3850
-	1    0    0    -1
-$EndComp
 Wire Wire Line
 	8800 4200 8800 4000
@@
 Wire Wire Line
 	5900 3850 5900 3800
+$Comp
+L D D5
+U 1 1 59E7AFF9
+P 8800 3850
+F 0 "D5" H 8800 3634 50  0000 C CNN
+F 1 "1N4148" H 8800 3725 50  0000 C CNN
+F 2 "" H 3050 2250 50  0001 C CNN
+F 3 "" H 3050 2250 50  0001 C CNN
+	1    8800 3850
+	0    -1   -1   0
+$EndComp
 $EndSCHEMATC
