File: SCH_PCB/CANDY/OZDUAL03A_01/SCH_PCB/OZDUAL03B.sch (KiCad schematic (older format))
At the start: 55 parts, among them J1 JUMP2_2x1, J2 POWER, J3 OPAMPA, J4 OPAMPB, J5 SOT23-6, M1 HOLE, M2 HOLE, M3 HOLE, M4 HOLE, Q1 BC846, U1 OZ, U2 MAX6066, U3 ANALOG SWITCH

Commit message: Data editing
update schema, new label
Parts:
- removed Q1: BC846, SOT-23-3, symbol BC849
- removed U2: MAX6066, SOT-23-3, symbol ISL21070CIH320Z-TK
- removed U3: ANALOG SWITCH, Mlab_IO:SOT-23-6, symbol TS5A3159
- removed c4, c5: C, Mlab_R:SMD-0805, symbol C-RESCUE-OZDUAL03A
- removed d3, d6: R, Mlab_R:SMD-0805, symbol R
- added C5, C6: C, Mlab_R:SMD-0805-hand-soldering, symbol C-RESCUE-OZDUAL03A
- added D4: 4k7R, Mlab_R:SMD-0805-hand-soldering, symbol R
- added D7: 0R, Mlab_R:SMD-0805-hand-soldering, symbol R
- added U2: LM4041AIM3-1,2V, Mlab_IO:SOT-23-6, symbol sot23-6
- A1: renamed from a0; value C -> 1uF; footprint Mlab_R:SMD-0805 -> Mlab_R:SMD-0805-hand-soldering
- A10: renamed from a9; value C -> 0R; footprint Mlab_R:SMD-0805 -> Mlab_R:SMD-0805-hand-soldering
- A2: renamed from a1; value R -> 10MR; footprint Mlab_R:SMD-0805 -> Mlab_R:SMD-0805-hand-soldering
- A3: renamed from a2; footprint Mlab_R:SMD-0805 -> Mlab_R:SMD-0805-hand-soldering
- A4: renamed from a3; footprint Mlab_R:SMD-0805 -> Mlab_R:SMD-0805-hand-soldering
- A5: renamed from a4; value C -> 1pF; footprint Mlab_R:SMD-0805 -> Mlab_R:SMD-0805-hand-soldering
- A6: renamed from a5; footprint Mlab_R:SMD-0805 -> Mlab_R:SMD-0805-hand-soldering
- A7: renamed from a6; footprint Mlab_R:SMD-0805 -> Mlab_R:SMD-0805-hand-soldering
- A8: renamed from a7; footprint Mlab_R:SMD-0805 -> Mlab_R:SMD-0805-hand-soldering
- A9: renamed from a8; value R -> 22kR; footprint Mlab_R:SMD-0805 -> Mlab_R:SMD-0805-hand-soldering
- B1: renamed from b0; value C -> 0R; footprint Mlab_R:SMD-0805 -> Mlab_R:SMD-0805-hand-soldering
- B10: renamed from b9; footprint Mlab_R:SMD-0805 -> Mlab_R:SMD-0805-hand-soldering
- B2: renamed from b1; value R -> 0R; footprint Mlab_R:SMD-0805 -> Mlab_R:SMD-0805-hand-soldering
- B3: renamed from b2; footprint Mlab_R:SMD-0805 -> Mlab_R:SMD-0805-hand-soldering
- B8: renamed from b7; value C -> 2n2F; footprint Mlab_R:SMD-0805 -> Mlab_R:SMD-0805-hand-soldering
- B9: renamed from b8; footprint Mlab_R:SMD-0805 -> Mlab_R:SMD-0805-hand-soldering
- C1: renamed from c1; footprint Mlab_R:SMD-0805 -> Mlab_R:SMD-0805-hand-soldering
- C10: renamed from c7; value C -> 0R; footprint Mlab_R:SMD-0805 -> Mlab_R:SMD-0805-hand-soldering
- C2: renamed from c0; value C -> 4u7F; footprint Mlab_R:SMD-0805 -> Mlab_R:SMD-0805-hand-soldering
- C3: renamed from c2; value R -> 0R; footprint Mlab_R:SMD-0805 -> Mlab_R:SMD-0805-hand-soldering
- C4: renamed from c3; value 100nF -> 0R; footprint Mlab_R:SMD-0805 -> Mlab_R:SMD-0805-hand-soldering
- C7: renamed from c6; value R -> 3k3R; footprint Mlab_R:SMD-0805 -> Mlab_R:SMD-0805-hand-soldering
- C8: renamed from c8; value R -> 1kR; footprint Mlab_R:SMD-0805 -> Mlab_R:SMD-0805-hand-soldering
- C9: renamed from c9; footprint Mlab_R:SMD-0805 -> Mlab_R:SMD-0805-hand-soldering
- Con2: renamed from C2; value 47u -> -
- Con4: renamed from C4; value 47u -> -
- D1: renamed from d0; footprint Mlab_R:SMD-0805 -> Mlab_R:SMD-0805-hand-soldering
- D10: renamed from d9; footprint Mlab_R:SMD-0805 -> Mlab_R:SMD-0805-hand-soldering
- D2: renamed from d1; footprint Mlab_R:SMD-0805 -> Mlab_R:SMD-0805-hand-soldering
- D3: renamed from d2; footprint Mlab_R:SMD-0805 -> Mlab_R:SMD-0805-hand-soldering
- D8: renamed from d7; value R -> 4u7F; footprint Mlab_R:SMD-0805 -> Mlab_R:SMD-0805-hand-soldering
- D9: renamed from d8; value R -> 0R; footprint Mlab_R:SMD-0805 -> Mlab_R:SMD-0805-hand-soldering
- Di2: renamed from D2; value M4 -> -
- R1: value R -> 100R; footprint Mlab_R:SMD-0805 -> Mlab_R:SMD-0805-hand-soldering
- R2: footprint Mlab_R:SMD-0805 -> Mlab_R:SMD-0805-hand-soldering
- U1: value OZ -> OPA2314
- renumbered C1 to Con1, C3 to Con3, D1 to Di1
Connections:
- net 1: now also C5.1, U2.1
- net 2: now also D4.2, U2.2
- net 3: now also C6.2, U2.3
- net 4: now also U2.4
- net 5: now also C5.2, C6.1, U2.5
- net 6: now also D7.1, U2.6
- net GNDA: now also D7.2
- net VCC: now also D4.1
Other:
- note added: "3V"
- note added: "A"
- note added: "CR2032"
- note added: "K"
- note added: "OUT TO OZDUAL03B_2"
- note added: "PIN DIODA"
- note added: "REF"
- note removed: "POWER INPUT"
- note removed: "REFERENCE, TRANSISTOR, SWITCH, ... in SOT23-3,5,6"

Commit message: Edit schema
Parts:
- A3, A7, B10, C1, C5, C6, C9: value C -> -
- A4, A8, B3, B9, D1, D10, D2, D3, R2: value R -> -
Changed lines of the file:
@@
 P 3100 1450
 F 0 "A4" V 3180 1450 50  0000 C CNN
-F 1 "R" V 3100 1450 50  0000 C CNN
+F 1 "-" V 3100 1450 50  0000 C CNN
 F 2 "Mlab_R:SMD-0805-hand-soldering" V 3030 1450 50  0001 C CNN
 F 3 "" H 3100 1450 50  0000 C CNN
@@
 P 2500 1700
 F 0 "D2" V 2580 1700 50  0000 C CNN
-F 1 "R" V 2500 1700 50  0000 C CNN
+F 1 "-" V 2500 1700 50  0000 C CNN
 F 2 "Mlab_R:SMD-0805-hand-soldering" V 2430 1700 50  0001 C CNN
 F 3 "" H 2500 1700 50  0000 C CNN
@@
 P 2250 1450
 F 0 "D1" V 2330 1450 50  0000 C CNN
-F 1 "R" V 2250 1450 50  0000 C CNN
+F 1 "-" V 2250 1450 50  0000 C CNN
 F 2 "Mlab_R:SMD-0805-hand-soldering" V 2180 1450 50  0001 C CNN
 F 3 "" H 2250 1450 50  0000 C CNN
@@
 P 2500 2700
 F 0 "D3" V 2580 2700 50  0000 C CNN
-F 1 "R" V 2500 2700 50  0000 C CNN
+F 1 "-" V 2500 2700 50  0000 C CNN
 F 2 "Mlab_R:SMD-0805-hand-soldering" V 2430 2700 50  0001 C CNN
 F 3 "" H 2500 2700 50  0000 C CNN
@@
 P 1800 1450
 F 0 "C1" H 1825 1550 50  0000 L CNN
-F 1 "C" H 1825 1350 50  0000 L CNN
+F 1 "-" H 1825 1350 50  0000 L CNN
 F 2 "Mlab_R:SMD-0805-hand-soldering" H 1838 1300 50  0001 C CNN
 F 3 "" H 1800 1450 50  0000 C CNN
@@
 P 3100 1150
 F 0 "A3" H 3125 1250 50  0000 L CNN
-F 1 "C" H 3125 1050 50  0000 L CNN
+F 1 "-" H 3125 1050 50  0000 L CNN
 F 2 "Mlab_R:SMD-0805-hand-soldering" H 3138 1000 50  0001 C CNN
 F 3 "" H 3100 1150 50  0000 C CNN
@@
 P 3100 4900
 F 0 "A8" V 3180 4900 50  0000 C CNN
-F 1 "R" V 3100 4900 50  0000 C CNN
+F 1 "-" V 3100 4900 50  0000 C CNN
 F 2 "Mlab_R:SMD-0805-hand-soldering" V 3030 4900 50  0001 C CNN
 F 3 "" H 3100 4900 50  0000 C CNN
@@
 P 2500 6150
 F 0 "D10" V 2580 6150 50  0000 C CNN
-F 1 "R" V 2500 6150 50  0000 C CNN
+F 1 "-" V 2500 6150 50  0000 C CNN
 F 2 "Mlab_R:SMD-0805-hand-soldering" V 2430 6150 50  0001 C CNN
 F 3 "" H 2500 6150 50  0000 C CNN
@@
 P 2250 6700
 F 0 "B9" V 2330 6700 50  0000 C CNN
-F 1 "R" V 2250 6700 50  0000 C CNN
+F 1 "-" V 2250 6700 50  0000 C CNN
 F 2 "Mlab_R:SMD-0805-hand-soldering" V 2180 6700 50  0001 C CNN
 F 3 "" H 2250 6700 50  0000 C CNN
@@
 P 3100 4650
 F 0 "A7" H 3125 4750 50  0000 L CNN
-F 1 "C" H 3125 4550 50  0000 L CNN
+F 1 "-" H 3125 4550 50  0000 L CNN
 F 2 "Mlab_R:SMD-0805-hand-soldering" H 3138 4500 50  0001 C CNN
 F 3 "" H 3100 4650 50  0000 C CNN
@@
 P 1800 6700
 F 0 "B10" H 1825 6800 50  0000 L CNN
-F 1 "C" H 1825 6600 50  0000 L CNN
+F 1 "-" H 1825 6600 50  0000 L CNN
 F 2 "Mlab_R:SMD-0805-hand-soldering" H 1838 6550 50  0001 C CNN
 F 3 "" H 1800 6700 50  0000 C CNN
@@
 P 2200 2450
 F 0 "B3" V 2280 2450 50  0000 C CNN
-F 1 "R" V 2200 2450 50  0000 C CNN
+F 1 "-" V 2200 2450 50  0000 C CNN
 F 2 "Mlab_R:SMD-0805-hand-soldering" V 2130 2450 50  0001 C CNN
 F 3 "" H 2200 2450 50  0000 C CNN
@@
 P 7050 2150
 F 0 "R2" V 7130 2150 50  0000 C CNN
-F 1 "R" V 7050 2150 50  0000 C CNN
+F 1 "-" V 7050 2150 50  0000 C CNN
 F 2 "Mlab_R:SMD-0805-hand-soldering" V 6980 2150 50  0001 C CNN
 F 3 "" H 7050 2150 50  0000 C CNN
@@
 P 1650 6050
 F 0 "C9" H 1675 6150 50  0000 L CNN
-F 1 "C" H 1675 5950 50  0000 L CNN
+F 1 "-" H 1675 5950 50  0000 L CNN
 F 2 "Mlab_R:SMD-0805-hand-soldering" H 1688 5900 50  0001 C CNN
 F 3 "" H 1650 6050 50  0000 C CNN
@@
 P 7950 4250
 F 0 "C5" H 7975 4350 50  0000 L CNN
-F 1 "C" H 7975 4150 50  0000 L CNN
+F 1 "-" H 7975 4150 50  0000 L CNN
 F 2 "Mlab_R:SMD-0805-hand-soldering" H 7988 4100 50  0001 C CNN
 F 3 "" H 7950 4250 50  0000 C CNN
@@
 P 7950 5000
 F 0 "C6" H 7975 5100 50  0000 L CNN
-F 1 "C" H 7975 4900 50  0000 L CNN
+F 1 "-" H 7975 4900 50  0000 L CNN
 F 2 "Mlab_R:SMD-0805-hand-soldering" H 7988 4850 50  0001 C CNN
 F 3 "" H 7950 5000 50  0000 C CNN
