File: SCH_PCB/CANDY/OZDUAL03A_02/SCH_PCB/OZDUAL03B.kicad_pcb (KiCad board)
At the start: 2 copper layers, 40.1 x 40.1 mm, 53 parts, among them Con1 47u, Con2 47u, Con3 47u, Con4 47u, J1 JUMP2_2x1, J2 POWER, J3 OPAMPA, J4 OPAMPB, J5 SOT23-6, M1 HOLE, M2 HOLE, M3 HOLE, M4 HOLE, U1 OZ, U2 sot23-6

Commit message: Edit schema
Parts:
- A1: value C -> 1N4148
- A10, B1, C10: value C -> 0R
- A2, A4, A8, B3, B9, C8, D1, D10, D2, D3, D4, R2: value R -> -
- A3, A5, A7, B10, B8, C1, C2, C6, C9: value C -> -
- A9, C3, D7: value R -> 0R
- B2: value R -> 1kR
- C4: value 100nF -> 0R
- C5: value C -> 10kR
- C7: value R -> 51R
- Con2, Con4: value 47u -> -
- D8: value R -> 1nF
- D9: value R -> 100R
- Di2: value M4 -> -
- R1: value R -> 10R
- U1: value OZ -> OPA2314
- U2: value sot23-6 -> BSS138

Commit message: Draw scheme
Parts:
- C5: value 10kR -> 120MR
- C7: value 51R -> 1N4148
Changed lines of the file:
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@@
       (effects (font (size 0.50038 0.50038) (thickness 0.10922)) (justify mirror))
     )
-    (fp_text value 10kR (at 0.127 -0.381 270) (layer B.SilkS)
+    (fp_text value 120MR (at 0.127 -0.381 270) (layer B.SilkS)
       (effects (font (size 0.50038 0.50038) (thickness 0.10922)) (justify mirror))
     )
@@
       (effects (font (size 0.50038 0.50038) (thickness 0.10922)) (justify mirror))
     )
-    (fp_text value 51R (at 0.127 -0.381 270) (layer B.SilkS)
+    (fp_text value 1N4148 (at 0.127 -0.381 270) (layer B.SilkS)
       (effects (font (size 0.50038 0.50038) (thickness 0.10922)) (justify mirror))
     )
